File: binary_clock/kicad/binaryclock.sch (KiCad schematic (older format))
At the start: 21 parts, among them U0 NodeMCU1.0(ESP-12E)

Commit message: D1 mini (Closes #1) (#2)
* Modifying code to use the D1 Mini board
* Updating schematic
Parts:
- removed U0: NodeMCU1.0(ESP-12E), symbol NodeMCU1.0(ESP-12E)
- added U1: WeMos_mini, symbol WeMos_mini
Connections:
- net at LED0.3 (GND), LED1.3 (GND), LED10.3 (GND)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: now also U1.2 (GND)
- net at LED0.4 (DIN): now also U1.3 (D4)
Changed lines of the file:
@@
 LIBS:ESP8266
 LIBS:ws2812b
+LIBS:wemos_mini
+LIBS:binaryclock-cache
 EELAYER 25 0
 EELAYER END
@@
 Title "Binary Clock"
 Date "2019-08-05"
-Rev "1.0"
+Rev "1.1"
 Comp ""
 Comment1 ""
@@
 Comment4 "Author: Patrick Connelly"
 $EndDescr
-$Comp
-L NodeMCU1.0(ESP-12E) U0
-U 1 1 5D4479AA
-P 10200 4300
-F 0 "U0" H 10200 5150 60  0000 C CNN
-F 1 "NodeMCU1.0(ESP-12E)" H 10200 3450 60  0000 C CNN
-F 2 "" H 9600 3450 60  0000 C CNN
-F 3 "" H 9600 3450 60  0000 C CNN
-	1    10200 4300
-	-1   0    0    1
-$EndComp
 $Comp
 L WS2812B LED0
@@
 	8900 4500 8600 4500
 Wire Wire Line
-	9400 4600 8900 4600
+	9200 4600 8900 4600
 Wire Wire Line
 	8900 4600 8900 5500
@@
 	9400 3700 9100 3700
 Wire Wire Line
-	9100 3700 9100 5600
-Wire Wire Line
-	9100 5600 600  5600
+	9100 5600 9100 3700
+Wire Wire Line
+	600  5600 9100 5600
 Wire Wire Line
 	8200 5600 8200 5500
@@
 Wire Wire Line
 	1900 1900 2300 1900
+$Comp
+L WeMos_mini U1
+U 1 1 5DA36BC1
+P 9900 3950
+F 0 "U1" H 9900 4450 60  0000 C CNN
+F 1 "WeMos_mini" H 9900 3450 60  0000 C CNN
+F 2 "" H 10450 3250 60  0000 C CNN
+F 3 "" H 10450 3250 60  0000 C CNN
+	1    9900 3950
+	1    0    0    -1
+$EndComp
+Wire Wire Line
+	9200 4600 9200 3800
+Wire Wire Line
+	9200 3800 9400 3800
 $EndSCHEMATC
